File: SimpleCart/SimpleCart.kicad_pcb (KiCad board)
At the start: 4 copper layers, 90 x 35.9 mm, 11 parts, among them J1 CommanderX16Expansion Alt, U1 SST39SF040 (ROM), U2 74HCT00, U3 74HCT138

Commit message: Laying the ground work (har har)
Routing:
- net GND: track 21.0 -> 20.0 mm, vias 42 -> 46
- net Net-(J1-A15): track 48.7 -> 49.7 mm
